File: A1301EUA-T_HallEffectBoard.kicad_pcb (KiCad board)
At the start: 2 copper layers, 21.6 x 27.9 mm, 6 parts, among them J1 Conn_01x03, U1 A1301EUA-T

Commit message: submitted to JLCPCB
Routing:
- net Net-(R2-Pad2): track 0.00 -> 17.7 mm
- net 5V_HALL_OUTPUT: track 17.6 -> 25.4 mm
Changed lines of the file:
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@@
       (layerselection 0x00010fc_ffffffff)
       (disableapertmacros false)
-      (usegerberextensions false)
+      (usegerberextensions true)
       (usegerberattributes true)
-      (usegerberadvancedattributes true)
-      (creategerberjobfile true)
+      (usegerberadvancedattributes false)
+      (creategerberjobfile false)
       (svguseinch false)
       (svgprecision 6)
@@
       (plotinvisibletext false)
       (sketchpadsonfab false)
-      (subtractmaskfromsilk false)
+      (subtractmaskfromsilk true)
       (outputformat 1)
       (mirror false)
-      (drillshape 1)
+      (drillshape 0)
       (scaleselection 1)
-      (outputdirectory "")
+      (outputdirectory "C:/Users/logans/OneDrive - PING/desktop/PROJ_KICAD/A1301EUA-T_HallEffectBoard/A1301EUA-T_HallEffectBoard/JLCPCB_OUTPUTS_6-23-2022/")
     )
   )
@@
   (segment (start 3.81 20.28) (end 3.81 16.51) (width 1) (layer "F.Cu") (net 1))
   (segment (start 12.74 21.59) (end 8.93 25.4) (width 1) (layer "F.Cu") (net 1))
+  (segment (start 18.3896 18.6944) (end 18.3896 16.51) (width 1) (layer "F.Cu") (net 1))
   (segment (start 13.97 21.59) (end 12.74 21.59) (width 1) (layer "F.Cu") (net 1))
+  (segment (start 15.494 21.59) (end 18.3896 18.6944) (width 1) (layer "F.Cu") (net 1))
+  (segment (start 13.97 21.59) (end 15.494 21.59) (width 1) (layer "F.Cu") (net 1))
   (segment (start 8.89 6.35) (end 13.97 6.35) (width 1) (layer "F.Cu") (net 3))
   (segment (start 8.89 6.35) (end 5.08 6.35) (width 1) (layer "F.Cu") (net 3))
@@
   (segment (start 5.08 6.35) (end 3.81 7.62) (width 1) (layer "F.Cu") (net 3))
   (segment (start 8.89 6.35) (end 8.89 2.54) (width 1) (layer "F.Cu") (net 3))
+  (segment (start 8.89 14.732) (end 12.192 11.43) (width 1) (layer "F.Cu") (net 4))
+  (segment (start 8.89 21.59) (end 8.89 14.732) (width 1) (layer "F.Cu") (net 4))
+  (segment (start 12.192 11.43) (end 18.3896 11.43) (width 1) (layer "F.Cu") (net 4))
   (zone (net 2) (net_name "GND") (layer "B.Cu") (hatch edge 0.508)
     (connect_pads (clearance 0.508))
